File: CANCap/CANCap.kicad_sch (KiCad schematic)
At the start: 5 parts, among them J1 M12x5 A-Type

Commit message: Misc. Tweaks to files
Other:
- moved on the sheet: J1
Changed lines of the file:
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@@
 	(wire
 		(pts
-			(xy 86.36 95.25) (xy 86.36 97.79)
+			(xy 88.9 93.98) (xy 88.9 96.52)
 		)
 		(stroke
@@
 	(wire
 		(pts
-			(xy 80.01 102.87) (xy 86.36 102.87)
-		)
-		(stroke
-			(width 0)
-			(type default)
-		)
-	)
-	(wire
-		(pts
-			(xy 80.01 100.33) (xy 93.98 100.33)
-		)
-		(stroke
-			(width 0)
-			(type default)
-		)
-	)
-	(wire
-		(pts
-			(xy 86.36 97.79) (xy 80.01 97.79)
+			(xy 82.55 101.6) (xy 88.9 101.6)
+		)
+		(stroke
+			(width 0)
+			(type default)
+		)
+	)
+	(wire
+		(pts
+			(xy 82.55 99.06) (xy 96.52 99.06)
+		)
+		(stroke
+			(width 0)
+			(type default)
+		)
+	)
+	(wire
+		(pts
+			(xy 88.9 96.52) (xy 82.55 96.52)
 		)
 		(stroke
@@
 	(wire
 		(pts
-			(xy 80.01 105.41) (xy 93.98 105.41)
+			(xy 82.55 104.14) (xy 96.52 104.14)
 		)
 		(stroke
@@
 	(wire
 		(pts
-			(xy 86.36 102.87) (xy 86.36 110.49)
+			(xy 88.9 101.6) (xy 88.9 109.22)
 		)
 		(stroke
@@
 	(wire
 		(pts
-			(xy 80.01 107.95) (xy 93.98 107.95)
+			(xy 82.55 106.68) (xy 96.52 106.68)
 		)
 		(stroke
@@
 	)
 	(label "CANH"
-		(at 93.98 100.33 180)
+		(at 96.52 99.06 180)
 		(effects
 			(font
@@
 	)
 	(label "CANL"
-		(at 93.98 105.41 180)
+		(at 96.52 104.14 180)
 		(effects
 			(font
@@
 	)
 	(label "ALERT"
-		(at 93.98 107.95 180)
+		(at 96.52 106.68 180)
 		(effects
 			(font
@@
 	(symbol
 		(lib_id "power:GND")
-		(at 86.36 110.49 0)
+		(at 88.9 109.22 0)
 		(unit 1)
 		(exclude_from_sim no)
@@
 		(fields_autoplaced yes)
 		(property "Reference" "#PWR01"
-			(at 86.36 116.84 0)
+			(at 88.9 115.57 0)
 			(effects
 				(font
@@
 		)
 		(property "Value" "GND"
-			(at 86.36 115.57 0)
+			(at 88.9 114.3 0)
 			(effects
 				(font
@@
 		)
 		(property "Footprint" ""
-			(at 86.36 110.49 0)
+			(at 88.9 109.22 0)
 			(effects
 				(font
@@
 		)
 		(property "Datasheet" ""
-			(at 86.36 110.49 0)
+			(at 88.9 109.22 0)
 			(effects
 				(font
@@
 		)
 		(property "Description" "Power symbol creates a global label with name \"GND\" , ground"
-			(at 86.36 110.49 0)
+			(at 88.9 109.22 0)
 			(effects
 				(font
@@
 	(symbol
 		(lib_id "Connector:Conn_01x05_Pin")
-		(at 74.93 102.87 0)
+		(at 77.47 101.6 0)
 		(unit 1)
 		(exclude_from_sim no)
@@
 		(fields_autoplaced yes)
 		(property "Reference" "J1"
-			(at 75.565 92.71 0)
+			(at 78.105 91.44 0)
 			(effects
 				(font
@@
 		)
 		(property "Value" "M12x5 A-Type"
-			(at 75.565 95.25 0)
+			(at 78.105 93.98 0)
 			(effects
 				(font
@@
 		)
 		(property "Footprint" "Extra_Footprints:M12x5_A_Circular_Connector"
-			(at 74.93 102.87 0)
+			(at 77.47 101.6 0)
 			(effects
 				(font
@@
 		)
 		(property "Datasheet" "~"
-			(at 74.93 102.87 0)
+			(at 77.47 101.6 0)
 			(effects
 				(font
@@
 		)
 		(property "Description" "Generic connector, single row, 01x05, script generated"
-			(at 74.93 102.87 0)
+			(at 77.47 101.6 0)
 			(effects
 				(font
@@
 	(symbol
 		(lib_id "power:+5V")
-		(at 86.36 95.25 0)
+		(at 88.9 93.98 0)
 		(unit 1)
 		(exclude_from_sim no)
@@
 		(fields_autoplaced yes)
 		(property "Reference" "#PWR02"
-			(at 86.36 99.06 0)
+			(at 88.9 97.79 0)
 			(effects
 				(font
@@
 		)
 		(property "Value" "+5V"
-			(at 86.36 90.17 0)
+			(at 88.9 88.9 0)
 			(effects
 				(font
@@
 		)
 		(property "Footprint" ""
-			(at 86.36 95.25 0)
+			(at 88.9 93.98 0)
 			(effects
 				(font
@@
 		)
 		(property "Datasheet" ""
-			(at 86.36 95.25 0)
+			(at 88.9 93.98 0)
 			(effects
 				(font
@@
 		)
 		(property "Description" "Power symbol creates a global label with name \"+5V\""
-			(at 86.36 95.25 0)
-			(effects
-				(font
+			(at 88.9 93.98 0)
+			(effects
+				(font
