File: CapstonePractice/CapstonePractice.kicad_pcb (KiCad board)
At the start: 4 copper layers, 53 x 47.4 mm, 35 parts, among them J2 M12x5 A-Type, J3 2x3 Header, J4 M12x5 A-Type, Q1 DMN2310U, U1 STM32F103C8Tx, U2 ATA6563, U4 TLV7xx_SOT23-5, Y1 8MHz 16pF Load

Commit message: Misc. Tweaks to files
Other:
- board size 53 x 47.4 mm -> 34.5 x 47.4 mm
Changed lines of the file:
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@@
 	)
 	(gr_rect
-		(start 120 63.2)
+		(start 138.5 63.2)
 		(end 173 110.6)
 		(stroke
