File: CapstonePractice/CapstonePractice.kicad_sch (KiCad schematic)
At the start: 29 parts, among them J2 M12x5 A-Type, J3 2x3 Header, J4 M12x5 A-Type, Q1 DMN2310U, U1 STM32F103C8Tx, U4 TLV7xx_SOT23-5, Y1 8MHz 16pF Load

Commit message: Misc. Tweaks to files
Other:
- moved on the sheet: C10, C5, C6, C7, C9, FB2, U1
