File: SensorCore_v1/SD_Card.kicad_sch (KiCad schematic)
At the start: 5 parts, among them J1 Micro_SD_Card_Det1, U4 EMIF06-MSD02N16

Commit message: Misc. Tweaks to files
Parts:
- removed C13: 10uF 16V, Capacitor_SMD:C_0805_2012Metric_Pad1.18x1.45mm_HandSolder, symbol Device:C
Other:
- moved on the sheet: C11, C3
Changed lines of the file:
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@@
 	(paper "A4")
 	(junction
-		(at 149.86 66.04)
-		(diameter 0)
-		(color 0 0 0 0)
-	)
-	(junction
-		(at 161.29 58.42)
-		(diameter 0)
-		(color 0 0 0 0)
-	)
-	(junction
-		(at 170.18 58.42)
+		(at 152.4 66.04)
 		(diameter 0)
 		(color 0 0 0 0)
@@
 	)
 	(junction
-		(at 161.29 66.04)
+		(at 152.4 58.42)
 		(diameter 0)
 		(color 0 0 0 0)
@@
 	(wire
 		(pts
-			(xy 161.29 66.04) (xy 170.18 66.04)
-		)
-		(stroke
-			(width 0)
-			(type default)
-		)
-	)
-	(wire
-		(pts
-			(xy 149.86 58.42) (xy 161.29 58.42)
+			(xy 152.4 58.42) (xy 163.83 58.42)
 		)
 		(stroke
@@
 	(wire
 		(pts
-			(xy 161.29 66.04) (xy 149.86 66.04)
+			(xy 163.83 66.04) (xy 152.4 66.04)
 		)
 		(stroke
@@
 	(wire
 		(pts
-			(xy 170.18 55.88) (xy 170.18 58.42)
-		)
-		(stroke
-			(width 0)
-			(type default)
-		)
-	)
-	(wire
-		(pts
-			(xy 161.29 58.42) (xy 170.18 58.42)
+			(xy 152.4 52.07) (xy 152.4 58.42)
 		)
 		(stroke
@@
 	(symbol
 		(lib_id "power:+5V")
-		(at 170.18 55.88 0)
+		(at 152.4 52.07 0)
 		(unit 1)
 		(exclude_from_sim no)
@@
 		(fields_autoplaced yes)
 		(property "Reference" "#PWR033"
-			(at 170.18 59.69 0)
+			(at 152.4 55.88 0)
 			(effects
 				(font
@@
 		)
 		(property "Value" "+3V3"
-			(at 170.18 50.8 0)
+			(at 152.4 46.99 0)
 			(effects
 				(font
@@
 		)
 		(property "Footprint" ""
-			(at 170.18 55.88 0)
+			(at 152.4 52.07 0)
 			(effects
 				(font
@@
 		)
 		(property "Datasheet" ""
-			(at 170.18 55.88 0)
+			(at 152.4 52.07 0)
 			(effects
 				(font
@@
 		)
 		(property "Description" "Power symbol creates a global label with name \"+5V\""
-			(at 170.18 55.88 0)
+			(at 152.4 52.07 0)
 			(effects
 				(font
@@
 				(path "/7f033487-c793-47e5-80dd-4bcaea87e7a6/48101682-9058-4889-ac83-741cfcdd5dc5"
 					(reference "#PWR033")
-					(unit 1)
-				)
-			)
-		)
-	)
-	(symbol
-		(lib_id "Device:C")
-		(at 170.18 62.23 0)
-		(unit 1)
-		(exclude_from_sim no)
-		(in_bom yes)
-		(on_board yes)
-		(dnp no)
-		(property "Reference" "C13"
-			(at 169.164 67.818 0)
-			(effects
-				(font
-					(size 1.27 1.27)
-				)
-			)
-		)
-		(property "Value" "10uF 16V"
-			(at 169.164 70.358 0)
-			(effects
-				(font
-					(size 1.27 1.27)
-				)
-			)
-		)
-		(property "Footprint" "Capacitor_SMD:C_0805_2012Metric_Pad1.18x1.45mm_HandSolder"
-			(at 171.1452 66.04 0)
-			(effects
-				(font
-					(size 1.27 1.27)
-				)
-				(hide yes)
-			)
-		)
-		(property "Datasheet" "~"
-			(at 170.18 62.23 0)
-			(effects
-				(font
-					(size 1.27 1.27)
-				)
-				(hide yes)
-			)
-		)
-		(property "Description" "Unpolarized capacitor"
-			(at 170.18 62.23 0)
-			(effects
-				(font
-					(size 1.27 1.27)
-				)
-				(hide yes)
-			)
-		)
-		(property "Digikey Part" "CL21A106KOQNNNE"
-			(at 170.18 62.23 0)
-			(effects
-				(font
-					(size 1.27 1.27)
-				)
-				(hide yes)
-			)
-		)
-		(pin "1"
-		)
-		(pin "2"
-		)
-		(instances
-			(project "SensorCore_v1"
-				(path "/7f033487-c793-47e5-80dd-4bcaea87e7a6/48101682-9058-4889-ac83-741cfcdd5dc5"
-					(reference "C13")
 					(unit 1)
 				)
@@
 	(symbol
 		(lib_id "power:GND")
-		(at 149.86 66.04 0)
+		(at 152.4 66.04 0)
 		(unit 1)
 		(exclude_from_sim no)
@@
 		(fields_autoplaced yes)
 		(property "Reference" "#PWR032"
-			(at 149.86 72.39 0)
+			(at 152.4 72.39 0)
 			(effects
 				(font
@@
 		)
 		(property "Value" "GND"
-			(at 149.86 71.12 0)
+			(at 152.4 71.12 0)
 			(effects
 				(font
@@
 		)
 		(property "Footprint" ""
-			(at 149.86 66.04 0)
+			(at 152.4 66.04 0)
 			(effects
 				(font
@@
 		)
 		(property "Datasheet" ""
-			(at 149.86 66.04 0)
+			(at 152.4 66.04 0)
 			(effects
 				(font
@@
 		)
 		(property "Description" "Power symbol creates a global label with name \"GND\" , ground"
-			(at 149.86 66.04 0)
+			(at 152.4 66.04 0)
 			(effects
 				(font
@@
 	(symbol
 		(lib_id "Device:C")
-		(at 149.86 62.23 180)
+		(at 152.4 62.23 180)
 		(unit 1)
 		(exclude_from_sim no)
@@
 		(dnp no)
 		(property "Reference" "C3"
-			(at 149.86 54.6099 0)
+			(at 152.4 54.6099 0)
 			(effects
 				(font
@@
 		)
 		(property "Value" "100nF"
-			(at 149.86 57.1499 0)
+			(at 152.4 57.1499 0)
 			(effects
 				(font
@@
 		)
 		(property "Footprint" "Resistor_SMD:R_0603_1608Metric_Pad0.98x0.95mm_HandSolder"
-			(at 148.8948 58.42 0)
+			(at 151.4348 58.42 0)
 			(effects
 				(font
@@
 		)
 		(property "Datasheet" "~"
-			(at 149.86 62.23 0)
+			(at 152.4 62.23 0)
 			(effects
 				(font
@@
 		)
 		(property "Description" "Unpolarized capacitor"
-			(at 149.86 62.23 0)
+			(at 152.4 62.23 0)
 			(effects
 				(font
@@
 		)
 		(property "Digikey Part" "CL10B104KB8NFNC"
-			(at 149.86 62.23 0)
+			(at 152.4 62.23 0)
 			(effects
 				(font
@@
 	(symbol
 		(lib_id "Device:C")
-		(at 161.29 62.23 0)
+		(at 163.83 62.23 0)
 		(unit 1)
 		(exclude_from_sim no)
@@
 		(dnp no)
 		(property "Reference" "C11"
-			(at 161.29 54.102 0)
+			(at 163.83 54.102 0)
 			(effects
 				(font
@@
 		)
 		(property "Value" "10uF 16V"
-			(at 161.29 56.642 0)
+			(at 163.83 56.642 0)
 			(effects
 				(font
@@
 		)
 		(property "Footprint" "Capacitor_SMD:C_0805_2012Metric_Pad1.18x1.45mm_HandSolder"
-			(at 162.2552 66.04 0)
+			(at 164.7952 66.04 0)
 			(effects
 				(font
@@
 		)
 		(property "Datasheet" "~"
-			(at 161.29 62.23 0)
+			(at 163.83 62.23 0)
 			(effects
 				(font
@@
 		)
 		(property "Description" "Unpolarized capacitor"
-			(at 161.29 62.23 0)
+			(at 163.83 62.23 0)
 			(effects
 				(font
@@
 		)
 		(property "Digikey Part" "CL21A106KOQNNNE"
-			(at 161.29 62.23 0)
-			(effects
-				(font
+			(at 163.83 62.23 0)
+			(effects
+				(font
