File: SensorCore_v1/SensorCore_v1.kicad_pcb (KiCad board)
At the start: 4 copper layers, 38 parts, among them J1 Micro_SD_Card_Det1, J2 M12x5 A-Type, J3 2x3 Header, J4 M12x5 A-Type, Q1 DMN2310U, U1 STM32C092KCT6, U2 ATA6563, U3 R-78K3.3-1.0, U4 EMIF06-MSD02N16, Y1 8MHz 16pF Load

Commit message: Misc. Tweaks to files
Parts:
- removed C13: 10uF 16V, Capacitor_SMD:C_0805_2012Metric_Pad1.18x1.45mm_HandSolder
- moved C3 4.39 mm to (154.3, 81.3), turned to -90 degrees
- moved C11 2.32 mm to (156.2, 81.1)
- moved U4 2.19 mm to (151.6, 81.2)
Routing:
- net GND: track 7.82 -> 13.0 mm
- net Net-(J1-DAT3/CD): track 6.11 -> 3.45 mm
- net Net-(J1-CMD): track 5.36 -> 2.83 mm
- net Net-(J1-DAT2): track 5.96 -> 4.05 mm
- net +3V3: track 11.4 -> 9.52 mm
- net Net-(J1-CLK): track 4.46 -> 2.83 mm
- net /SD_Card/Card Detect: track 8.93 -> 9.85 mm, vias 0 -> 2
- net Net-(J1-DAT0): track 5.30 -> 4.47 mm
