File: SensorCore_v1/SensorCore_v1.kicad_sch (KiCad schematic)
At the start: 18 parts, among them J2 M12x5 A-Type, J3 2x3 Header, J4 M12x5 A-Type, Q1 DMN2310U, U1 STM32C092KCT6, Y1 8MHz 16pF Load

Commit message: Misc. Tweaks to files
Parts:
- added C20, C21: 27pF, Capacitor_SMD:C_0603_1608Metric_Pad1.08x0.95mm_HandSolder, symbol Device:C
- added Y2: 8MHz 16pF Load, Extra_Footprints:Crystal_6x3.5mm, symbol Device:Crystal
Connections:
- net GND: now also C20.2, C21.2
- net OSC+: now also C20.1, Y2.1
- net OSC-: now also C21.1, Y2.2
Other:
- moved on the sheet: J3
